File: Files/CustomKB2040.kicad_pcb (KiCad board)
At the start: 4 copper layers, 225.2 x 105.2 mm, 161 parts, among them J1 USB_C_Receptacle, J3 USB_C_Receptacle, J4 USB_C_Receptacle, J5 Conn_01x03_Pin, J6 USB_C_Receptacle, U1 W25Q128JVS, U2 XC6206-3.3_SOT, U3 USBLC6-2SC6, U4 RP2040, U5 W25Q128JVS, U6 XC6206-3.3_SOT, U7 USBLC6-2SC6, U8 RP2040, Y1 Crystal_GND24, Y2 Crystal_GND24

Commit message: Finished left side
Parts:
- removed the D3 at (242.5, 101.0)
- removed the D4 at (242.5, 105.3)
- added D41: Placeholder_LED, ScottoKeebs_Components:LED_0805, F.Cu at (245.8, 65.2)
- added D42: Placeholder_LED, ScottoKeebs_Components:LED_0805, F.Cu at (245.8, 69.5)
- moved D1 86.0 mm to (192.5, 163.0), turned to -12 degrees
- moved C30 70.2 mm to (240.3, 40.8)
- moved S9 69.2 mm to (113.2, 101.4)
- moved D3 69.2 mm to (151.0, 158.6)
- moved D6 69.2 mm to (113.0, 134.9)
- moved D7 69.2 mm to (94.0, 139.6)
- moved D8 69.2 mm to (75.0, 151.5)
- moved D9 69.2 mm to (75.0, 132.5)
- moved S11 69.2 mm to (113.0, 139.6)
- moved S12 69.2 mm to (191.4, 168.1)
- moved S15 69.2 mm to (132.0, 144.4)
- moved S18 69.2 mm to (151.2, 144.4)
- moved S2 69.2 mm to (75.0, 137.2)
- moved S3 69.2 mm to (75.0, 156.2)
- moved S4 69.2 mm to (151.0, 163.4)
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- renumbered D5 to D1, D14 to D10, D15 to D11, D16 to D12, D17 to D13, D18 to D14, D19 to D15, D20 to D16, D21 to D17, D22 to D18, D1 to D19, D6 to D2, D2 to D20, D7 to D3, D8 to D4, D9 to D5, D10 to D6, D11 to D7, D12 to D8, D13 to D9
Connections:
- D1 pad 4: GPIO_0 -> GPIO_19_LEDS
- S11 pad 1: GPIO_13 -> GPIO_14
- S15 pad 1: GPIO_14 -> GPIO_13
- S18 pad 1: GPIO_15 -> GPIO_12
- S7 pad 1: GPIO_12 -> GPIO_15
- U4 pad 30: unconnected-(U4-GPIO19-Pad30) -> GPIO_19_LEDS
Routing:
- net +3V3: track 37.5 -> 120.3 mm, vias 7 -> 10
- net GPIO_15: track 16.6 -> 86.4 mm
- net GPIO_14: track 15.7 -> 68.2 mm
- net GPIO_18: track 0.00 -> 43.0 mm, vias 0 -> 1
- net GPIO_16: track 4.08 -> 44.8 mm, vias 0 -> 1
- net GPIO_17: track 2.66 -> 40.1 mm, vias 0 -> 1
- net Net-(D1-DOUT): track 0.00 -> 32.4 mm, vias 0 -> 2
- net GPIO_19_LEDS: track 0.00 -> 32.3 mm, vias 0 -> 1
- net GPIO_13: track 14.7 -> 46.1 mm
- net GPIO_25: track 1.18 -> 28.3 mm, vias 1 -> 2
- net GND: track 39.5 -> 64.6 mm, vias 35 -> 65
- net +1V1: track 13.7 -> 26.3 mm
- net GPIO_12: track 13.7 -> 24.3 mm
- net USB_BOOT: track 6.40 -> 8.36 mm
- net RESET: track 15.6 -> 16.9 mm
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Other:
- board size 225.2 x 105.2 mm -> 279.4 x 87.9 mm
- board text added: "Still working on this side"
