File: Files/Left_Side.kicad_sch (KiCad schematic)
At the start: 77 parts, among them J1 USB_C_Receptacle, J3 USB_C_Receptacle, U1 W25Q128JVS, U2 XC6206-3.3_SOT, U3 USBLC6-2SC6, U4 RP2040, Y1 Crystal_GND24

Commit message: Finished left side
Parts:
- renumbered D5 to D1, D14 to D10, D15 to D11, D16 to D12, D17 to D13, D18 to D14, D19 to D15, D20 to D16, D21 to D17, D22 to D18, D1 to D19, D6 to D2, D2 to D20, D7 to D3, D8 to D4, D9 to D5, D10 to D6, D11 to D7, D12 to D8, D13 to D9
Connections:
- net GPIO_0: no longer D1.4 (DIN)
- net GPIO_12: now also S18.1; no longer S7.1
- net GPIO_13: now also S15.1; no longer S11.1
- net GPIO_14: now also S11.1; no longer S15.1
- net GPIO_15: now also S7.1; no longer S18.1
- net GPIO_19_LEDS: now reaches U4.30 (GPIO19)
- net GPIO_19_LEDS: now also D1.4 (DIN)
- no-connect marks 33 -> 32
Changed lines of the file:
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@@
 	)
 	(no_connect
-		(at 240.03 134.62)
-	)
-	(no_connect
 		(at 240.03 139.7)
 	)
@@
 	(wire
 		(pts
-			(xy 33.02 24.13) (xy 33.02 27.94)
+			(xy 33.02 22.86) (xy 33.02 27.94)
 		)
 		(stroke
@@
 	(global_label "GPIO_15"
 		(shape input)
-		(at 364.49 130.81 180)
+		(at 306.07 130.81 180)
 		(fields_autoplaced yes)
 		(effects
@@
 		)
 		(property "Intersheetrefs" "${INTERSHEET_REFS}"
-			(at 353.6429 130.81 0)
+			(at 295.2229 130.81 0)
 			(effects
 				(font
@@
 	(global_label "GPIO_0"
 		(shape input)
-		(at 33.02 24.13 0)
-		(fields_autoplaced yes)
-		(effects
-			(font
-				(size 1.27 1.27)
-			)
-			(justify left)
-		)
-		(property "Intersheetrefs" "${INTERSHEET_REFS}"
-			(at 42.6576 24.13 0)
-			(effects
-				(font
-					(size 1.27 1.27)
-				)
-				(justify left)
-				(hide yes)
-			)
-		)
-	)
-	(global_label "GPIO_0"
-		(shape input)
 		(at 240.03 86.36 0)
 		(fields_autoplaced yes)
@@
 	(global_label "GPIO_12"
 		(shape input)
-		(at 306.07 130.81 180)
+		(at 364.49 130.81 180)
 		(fields_autoplaced yes)
 		(effects
@@
 		)
 		(property "Intersheetrefs" "${INTERSHEET_REFS}"
-			(at 295.2229 130.81 0)
+			(at 353.6429 130.81 0)
 			(effects
 				(font
@@
 		)
 	)
+	(global_label "GPIO_19_LEDS"
+		(shape input)
+		(at 33.02 22.86 0)
+		(fields_autoplaced yes)
+		(effects
+			(font
+				(size 1.27 1.27)
+			)
+			(justify left)
+		)
+		(property "Intersheetrefs" "${INTERSHEET_REFS}"
+			(at 49.4913 22.86 0)
+			(effects
+				(font
+					(size 1.27 1.27)
+				)
+				(justify left)
+				(hide yes)
+			)
+		)
+	)
 	(global_label "L_TX"
 		(shape input)
@@
 	(global_label "GPIO_13"
 		(shape input)
-		(at 325.12 130.81 180)
+		(at 344.17 130.81 180)
 		(fields_autoplaced yes)
 		(effects
@@
 		)
 		(property "Intersheetrefs" "${INTERSHEET_REFS}"
-			(at 314.2729 130.81 0)
+			(at 333.3229 130.81 0)
 			(effects
 				(font
@@
 		)
 	)
+	(global_label "GPIO_19_LEDS"
+		(shape input)
+		(at 240.03 134.62 0)
+		(fields_autoplaced yes)
+		(effects
+			(font
+				(size 1.27 1.27)
+			)
+			(justify left)
+		)
+		(property "Intersheetrefs" "${INTERSHEET_REFS}"
+			(at 256.5013 134.62 0)
+			(effects
+				(font
+					(size 1.27 1.27)
+				)
+				(justify left)
+				(hide yes)
+			)
+		)
+	)
 	(global_label "GPIO_6"
 		(shape input)
@@
 	(global_label "GPIO_14"
 		(shape input)
-		(at 344.17 130.81 180)
+		(at 325.12 130.81 180)
 		(fields_autoplaced yes)
 		(effects
@@
 		)
 		(property "Intersheetrefs" "${INTERSHEET_REFS}"
-			(at 333.3229 130.81 0)
+			(at 314.2729 130.81 0)
 			(effects
 				(font
@@
 		(on_board yes)
 		(dnp no)
-		(property "Reference" "D20"
+		(property "Reference" "D16"
 			(at 45.72 260.858 0)
 			(effects
@@
 			(project "CustomKB2040"
 				(path "/1dc59942-63a2-41f5-a9fb-7502b7672a2f/02cee8b0-a02f-4615-921b-eb372b3c289b"
-					(reference "D20")
+					(reference "D16")
 					(unit 1)
 				)
@@
 		(on_board yes)
 		(dnp no)
-		(property "Reference" "D7"
+		(property "Reference" "D3"
 			(at 43.942 66.04 90)
 			(effects
@@
 			(project "CustomKB2040"
 				(path "/1dc59942-63a2-41f5-a9fb-7502b7672a2f/02cee8b0-a02f-4615-921b-eb372b3c289b"
-					(reference "D7")
+					(reference "D3")
 					(unit 1)
 				)
@@
 		(on_board yes)
 		(dnp no)
-		(property "Reference" "D8"
+		(property "Reference" "D4"
 			(at 43.942 81.28 90)
 			(effects
@@
 			(project "CustomKB2040"
 				(path "/1dc59942-63a2-41f5-a9fb-7502b7672a2f/02cee8b0-a02f-4615-921b-eb372b3c289b"
-					(reference "D8")
+					(reference "D4")
 					(unit 1)
 				)
@@
 		(on_board yes)
 		(dnp no)
-		(property "Reference" "D16"
+		(property "Reference" "D12"
 			(at 43.942 203.2 90)
 			(effects
@@
 			(project "CustomKB2040"
 				(path "/1dc59942-63a2-41f5-a9fb-7502b7672a2f/02cee8b0-a02f-4615-921b-eb372b3c289b"
-					(reference "D16")
+					(reference "D12")
 					(unit 1)
 				)
@@
 		(on_board yes)
 		(dnp no)
-		(property "Reference" "D19"
+		(property "Reference" "D15"
 			(at 43.942 248.92 90)
 			(effects
@@
 			(project "CustomKB2040"
 				(path "/1dc59942-63a2-41f5-a9fb-7502b7672a2f/02cee8b0-a02f-4615-921b-eb372b3c289b"
-					(reference "D19")
+					(reference "D15")
 					(unit 1)
 				)
@@
 		(on_board yes)
 		(dnp no)
-		(property "Reference" "D12"
+		(property "Reference" "D8"
 			(at 43.942 142.24 90)
 			(effects
@@
 			(project "CustomKB2040"
 				(path "/1dc59942-63a2-41f5-a9fb-7502b7672a2f/02cee8b0-a02f-4615-921b-eb372b3c289b"
-					(reference "D12")
+					(reference "D8")
 					(unit 1)
 				)
@@
 		(on_board yes)
 		(dnp no)
-		(property "Reference" "D14"
+		(property "Reference" "D10"
 			(at 43.942 172.72 90)
 			(effects
@@
 			(project "CustomKB2040"
 				(path "/1dc59942-63a2-41f5-a9fb-7502b7672a2f/02cee8b0-a02f-4615-921b-eb372b3c289b"
-					(reference "D14")
+					(reference "D10")
 					(unit 1)
 				)
@@
 		(on_board yes)
 		(dnp no)
-		(property "Reference" "D9"
+		(property "Reference" "D5"
 			(at 43.942 96.52 90)
 			(effects
@@
 			(project "CustomKB2040"
 				(path "/1dc59942-63a2-41f5-a9fb-7502b7672a2f/02cee8b0-a02f-4615-921b-eb372b3c289b"
-					(reference "D9")
+					(reference "D5")
 					(unit 1)
 				)
@@
 		(dnp no)
 		(fields_autoplaced yes)
-		(property "Reference" "D1"
+		(property "Reference" "D19"
 			(at 186.69 216.2174 90)
 			(effects
@@
 			(project "CustomKB2040"
 				(path "/1dc59942-63a2-41f5-a9fb-7502b7672a2f/02cee8b0-a02f-4615-921b-eb372b3c289b"
-					(reference "D1")
+					(reference "D19")
 					(unit 1)
 				)
@@
 		(dnp no)
 		(fields_autoplaced yes)
-		(property "Reference" "D2"
+		(property "Reference" "D20"
 			(at 217.17 216.2174 90)
 			(effects
@@
 			(project "CustomKB2040"
 				(path "/1dc59942-63a2-41f5-a9fb-7502b7672a2f/02cee8b0-a02f-4615-921b-eb372b3c289b"
-					(reference "D2")
+					(reference "D20")
 					(unit 1)
 				)
@@
 		(on_board yes)
 		(dnp no)
-		(property "Reference" "D17"
+		(property "Reference" "D13"
 			(at 43.942 218.44 90)
 			(effects
@@
 			(project "CustomKB2040"
 				(path "/1dc59942-63a2-41f5-a9fb-7502b7672a2f/02cee8b0-a02f-4615-921b-eb372b3c289b"
-					(reference "D17")
+					(reference "D13")
 					(unit 1)
 				)
@@
 		(on_board yes)
 		(dnp no)
-		(property "Reference" "D13"
+		(property "Reference" "D9"
 			(at 43.942 157.48 90)
 			(effects
@@
 			(project "CustomKB2040"
 				(path "/1dc59942-63a2-41f5-a9fb-7502b7672a2f/02cee8b0-a02f-4615-921b-eb372b3c289b"
-					(reference "D13")
+					(reference "D9")
 					(unit 1)
 				)
@@
 		(on_board yes)
 		(dnp no)
-		(property "Reference" "D15"
+		(property "Reference" "D11"
 			(at 43.942 187.96 90)
 			(effects
@@
 			(project "CustomKB2040"
 				(path "/1dc59942-63a2-41f5-a9fb-7502b7672a2f/02cee8b0-a02f-4615-921b-eb372b3c289b"
-					(reference "D15")
+					(reference "D11")
 					(unit 1)
 				)
@@
 		(dnp no)
 		(fields_autoplaced yes)
-		(property "Reference" "D5"
+		(property "Reference" "D1"
 			(at 46.99 26.7014 90)
 			(effects
@@
 			(project ""
 				(path "/1dc59942-63a2-41f5-a9fb-7502b7672a2f/02cee8b0-a02f-4615-921b-eb372b3c289b"
-					(reference "D5")
+					(reference "D1")
 					(unit 1)
 				)
@@
 		(on_board yes)
 		(dnp no)
-		(property "Reference" "D6"
+		(property "Reference" "D2"
 			(at 43.942 50.8 90)
 			(effects
@@
 			(project "CustomKB2040"
 				(path "/1dc59942-63a2-41f5-a9fb-7502b7672a2f/02cee8b0-a02f-4615-921b-eb372b3c289b"
-					(reference "D6")
+					(reference "D2")
 					(unit 1)
 				)
@@
 		(on_board yes)
 		(dnp no)
-		(property "Reference" "D22"
+		(property "Reference" "D18"
 			(at 76.2 260.858 0)
 			(effects
@@
 			(project "CustomKB2040"
 				(path "/1dc59942-63a2-41f5-a9fb-7502b7672a2f/02cee8b0-a02f-4615-921b-eb372b3c289b"
-					(reference "D22")
+					(reference "D18")
 					(unit 1)
 				)
@@
 		(on_board yes)
 		(dnp no)
-		(property "Reference" "D10"
+		(property "Reference" "D6"
 			(at 43.942 111.76 90)
 			(effects
@@
 			(project "CustomKB2040"
 				(path "/1dc59942-63a2-41f5-a9fb-7502b7672a2f/02cee8b0-a02f-4615-921b-eb372b3c289b"
-					(reference "D10")
+					(reference "D6")
 					(unit 1)
 				)
@@
 		(on_board yes)
 		(dnp no)
-		(property "Reference" "D21"
+		(property "Reference" "D17"
 			(at 60.96 260.858 0)
 			(effects
@@
 			(project "CustomKB2040"
 				(path "/1dc59942-63a2-41f5-a9fb-7502b7672a2f/02cee8b0-a02f-4615-921b-eb372b3c289b"
-					(reference "D21")
+					(reference "D17")
 					(unit 1)
 				)
@@
 		(on_board yes)
 		(dnp no)
-		(property "Reference" "D11"
+		(property "Reference" "D7"
 			(at 43.942 127 90)
 			(effects
@@
 			(project "CustomKB2040"
 				(path "/1dc59942-63a2-41f5-a9fb-7502b7672a2f/02cee8b0-a02f-4615-921b-eb372b3c289b"
-					(reference "D11")
+					(reference "D7")
 					(unit 1)
 				)
@@
 		(on_board yes)
 		(dnp no)
-		(property "Reference" "D18"
+		(property "Reference" "D14"
 			(at 43.942 233.68 90)
 			(effects
@@
 			(project "CustomKB2040"
 				(path "/1dc59942-63a2-41f5-a9fb-7502b7672a2f/02cee8b0-a02f-4615-921b-eb372b3c289b"
-					(reference "D18")
+					(reference "D14")
 					(unit 1)
 				)
