File: PCBs/CustomKB2040.kicad_pcb (KiCad board)
At the start: 4 copper layers, 279.4 x 87.9 mm, 161 parts, among them J1 USB_C_Receptacle, J3 USB_C_Receptacle, J4 USB_C_Receptacle, J5 Conn_01x03_Pin, J6 USB_C_Receptacle, U1 W25Q128JVS, U2 XC6206-3.3_SOT, U3 USBLC6-2SC6, U4 RP2040, U5 W25Q128JVS, U6 XC6206-3.3_SOT, U7 USBLC6-2SC6, U8 RP2040, Y1 Crystal_GND24, Y2 Crystal_GND24

Commit message: store for replacement
Parts:
- removed J5: Conn_01x03_Pin, Connector_JST:JST_XH_B3B-XH-AM_1x03_P2.50mm_Vertical
- moved D23 181.3 mm to (354.8, 122.2)
- moved D24 181.3 mm to (354.8, 126.9)
- moved D25 181.3 mm to (354.8, 131.5)
- moved D26 181.3 mm to (354.8, 136.1)
- moved D27 181.3 mm to (354.8, 140.7)
- moved D28 181.3 mm to (354.8, 145.3)
- moved D29 181.3 mm to (354.8, 149.9)
- moved D30 181.3 mm to (362.6, 122.2)
- moved D31 181.3 mm to (362.6, 126.9)
- moved D32 181.3 mm to (362.6, 131.5)
- moved D33 181.3 mm to (362.6, 136.1)
- moved D34 181.3 mm to (362.6, 140.7)
- moved D35 181.3 mm to (362.6, 145.3)
- moved D36 181.3 mm to (362.6, 149.9)
- moved D37 181.3 mm to (370.4, 122.2)
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Routing:
- net GND: track 64.6 -> 68.6 mm, vias 65 -> 60
- removed copper zone on F.Cu, net GND
Other:
- board text removed: "Still working on this side"
