File: PCBs/CustomKB2040.kicad_pcb (KiCad board)
At the start: 4 copper layers, 278.9 x 87.9 mm, 167 parts, among them J1 USB_C_Receptacle, J3 USB_C_Receptacle, J4 USB_C_Receptacle, J6 USB_C_Receptacle, U1 W25Q128JVS, U2 XC6206-3.3_SOT, U3 USBLC6-2SC6, U4 RP2040, U5 W25Q128JVS, U6 XC6206-3.3_SOT, U7 USBLC6-2SC6, U8 RP2040, Y1 Crystal_GND24, Y2 Crystal_GND24

Commit message: mid way right side
Parts:
- added C38: 100n, Capacitor_SMD:C_0603_1608Metric, F.Cu at (228.0, 127.5)
- added REF**: Mouse_Bites_7, ScottoKeebs_Miscellaneous:Mouse_Bites_7, F.Cu at (142.4, 95.0)
- added REF**: Mouse_Bites_7, ScottoKeebs_Miscellaneous:Mouse_Bites_7, F.Cu at (185.5, 137.0)
- added REF**: Mouse_Bites_7, ScottoKeebs_Miscellaneous:Mouse_Bites_7, F.Cu at (266.5, 95.0)
- added REF**: Mouse_Bites_7, ScottoKeebs_Miscellaneous:Mouse_Bites_7, F.Cu at (113.2, 156.4)
- added REF**: Mouse_Bites_7, ScottoKeebs_Miscellaneous:Mouse_Bites_7, F.Cu at (293.9, 156.3)
- added REF**: Mouse_Bites_7, ScottoKeebs_Miscellaneous:Mouse_Bites_7, F.Cu at (222.9, 137.4)
- C25, C26, C31: moved to B.Cu
- moved C26 28.4 mm to (240.5, 129.8)
- moved C34 25.2 mm to (242.5, 132.9)
- moved C33 23.7 mm to (242.5, 134.4)
- moved C30 22.8 mm to (242.5, 131.4)
- moved C32 22.7 mm to (242.5, 136.9)
- moved C27 20.1 mm to (228.0, 130.5), turned to 180 degrees
- moved C25 19.6 mm to (235.5, 143.0), turned to -90 degrees
- moved C35 19.4 mm to (228.0, 129.0), turned to 180 degrees
- moved C31 18.2 mm to (237.0, 143.0), turned to -90 degrees
- moved C28 11.6 mm to (243.5, 116.5)
- moved U6 11.4 mm to (243.5, 110.5)
- moved C22 11.4 mm to (243.5, 113.5)
- moved C20 11.4 mm to (243.5, 108.0)
- moved C29 9.73 mm to (228.0, 137.0), turned to 180 degrees
- moved F2 9.00 mm to (243.5, 115.0), turned to 180 degrees
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Connections:
- net L_D+_R renamed L_R D+
- net L_D-_R renamed L_R D-
- J4 pad A6: USB D+_R -> USB_R D+
- J4 pad A7: USB D-_R -> USB_R D-
- J4 pad B6: USB D+_R -> USB_R D+
- J4 pad B7: USB D-_R -> USB_R D-
- R18 pad 2: Net-(U8-USB_DP) -> USB_R D+
- R19 pad 1: Net-(U8-USB_DM) -> USB_R D-
- U7 pad 3: USB D-_R -> USB_R D-
- U7 pad 4: USB D+_R -> USB_R D+
- U8 pad 46: Net-(U8-USB_DM) -> USB_R D-
- U8 pad 47: Net-(U8-USB_DP) -> USB_R D+
Routing:
- net +3V3_R: track 1.07 -> 37.7 mm, vias 1 -> 4
- net GND_R: track 7.27 -> 40.5 mm, vias 6 -> 27
- net L_R D+: track 0.00 -> 19.1 mm
- net L_R D-: track 0.00 -> 17.8 mm
- net +1V1_R: track 0.00 -> 13.5 mm, vias 0 -> 3
- net USB_R D+: track 0.00 -> 11.8 mm
- net USB_R D-: track 0.00 -> 10.5 mm
- net USB D+_R: track 9.42 -> 0.00 mm
- net Net-(U8-XIN): track 0.00 -> 9.20 mm
- net Net-(U8-XOUT): track 0.00 -> 8.63 mm
- net USB D-_R: track 8.11 -> 0.00 mm
- net RESET_R: track 0.00 -> 7.42 mm
- net USB_BOOT_R: track 0.00 -> 5.78 mm
- net Net-(U6-VO): track 0.00 -> 4.52 mm
- net Net-(C24-Pad1): track 0.00 -> 3.69 mm
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Other:
- board size 278.9 x 87.9 mm -> 278.9 x 107.1 mm

Commit message: edge outline done
Parts:
- moved REF** 100.3 mm to (94.0, 96.0), turned to -90 degrees
- moved REF** 100.1 mm to (314.0, 96.0), turned to -90 degrees
- moved C21 1.70 mm to (246.0, 128.4), turned to -90 degrees
- moved REF** 1.49 mm to (295.0, 155.3)
- moved REF** 1.12 mm to (266.0, 96.0)
- moved REF** 1.12 mm to (113.0, 155.3)
- moved R18 1.10 mm to (236.5, 128.4)
- moved R19 1.10 mm to (238.0, 128.4)
- moved REF** 1.08 mm to (142.0, 96.0)
Routing:
- net GPIO_0_R: track 0.00 -> 48.8 mm, vias 0 -> 1
- net +3V3_R: track 37.7 -> 84.3 mm, vias 4 -> 7
- net QSPI_SS_R: track 0.00 -> 23.6 mm, vias 0 -> 2
- net Net-(D29-DOUT): track 0.00 -> 23.1 mm
- net QSPI_SD1_R: track 0.00 -> 20.3 mm, vias 0 -> 2
- net Net-(D30-DOUT): track 0.00 -> 20.1 mm
- net Net-(D35-DOUT): track 0.00 -> 20.1 mm
- net Net-(D25-DOUT): track 0.00 -> 19.8 mm
- net QSPI_SD2_R: track 0.00 -> 18.9 mm, vias 0 -> 2
- net GND_R: track 40.5 -> 58.7 mm, vias 27 -> 47
- net Net-(D28-DOUT): track 0.00 -> 17.2 mm
- net Net-(D38-DOUT): track 0.00 -> 17.2 mm
- net Net-(D24-DOUT): track 0.00 -> 17.0 mm
- net Net-(D23-DOUT): track 0.00 -> 16.4 mm
- net Net-(D36-DOUT): track 0.00 -> 15.3 mm
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- added copper zone on F.Cu, net +3V3_R
Other:
- board size 278.9 x 107.1 mm -> 279 x 107 mm

Commit message: making progress
Parts:
- moved C25 4.00 mm to (239.5, 142.9)
- moved C31 1.01 mm to (238.0, 142.9)
- moved C23 0.96 mm to (233.1, 147.6)
- moved C24 0.96 mm to (235.6, 150.6)
- moved R16 0.96 mm to (238.1, 147.6)
- moved Y2 0.96 mm to (235.6, 147.6)
- moved R14 0.71 mm to (243.9, 103.2), turned to 0 degrees
- moved C29 0.67 mm to (227.4, 137.3), turned to -90 degrees
Connections:
- U8 pad 24: SWCLK_R -> unconnected-(U8-SWCLK-Pad24)
- U8 pad 25: SWD_R -> unconnected-(U8-SWD-Pad25)
Routing:
- net GPIO_5_R: track 0.00 -> 111.3 mm, vias 0 -> 1
- net GPIO_9_R: track 0.00 -> 97.8 mm, vias 0 -> 1
- net GPIO_14_R: track 0.00 -> 95.5 mm, vias 0 -> 1
- net GPIO_4_R: track 0.00 -> 74.0 mm, vias 0 -> 1
- net GPIO_13_R: track 0.00 -> 73.9 mm, vias 0 -> 1
- net GPIO_17_R: track 0.00 -> 69.5 mm
- net GPIO_3_R: track 0.00 -> 52.9 mm, vias 0 -> 1
- net GPIO_8_R: track 0.00 -> 51.3 mm, vias 0 -> 1
- net GPIO_16_R: track 0.00 -> 51.1 mm
- net GPIO_10_R: track 0.00 -> 42.3 mm
- net GPIO_18_R: track 0.00 -> 40.5 mm
- net QSPI_SS_R: track 23.6 -> 61.7 mm, vias 2 -> 3
- net GPIO_15_R: track 0.00 -> 36.6 mm
- net GPIO_11_R: track 0.00 -> 34.6 mm, vias 0 -> 2
- net Net-(D33-DOUT): track 0.00 -> 33.4 mm, vias 0 -> 2
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
Commit message: arragned right side
Parts:
- C27, C29, C30, C35, C36, C38: moved to B.Cu
- moved R13 24.3 mm to (226.3, 135.7), turned to 90 degrees
- moved C21 19.8 mm to (226.3, 130.7), turned to 90 degrees
- moved C31 19.3 mm to (247.1, 125.9), turned to 90 degrees
- moved C27 17.4 mm to (245.2, 127.7), turned to 90 degrees
- moved C29 16.0 mm to (243.3, 139.3)
- moved U5 14.6 mm to (230.3, 132.8), turned to 90 degrees
- moved C30 12.4 mm to (230.1, 131.3), turned to 180 degrees
- moved C32 12.4 mm to (238.7, 125.1), turned to 90 degrees
- moved C36 10.6 mm to (236.4, 138.4), turned to -90 degrees
- moved C33 9.53 mm to (240.4, 125.1), turned to 90 degrees
- moved C25 8.16 mm to (235.8, 135.6), turned to 180 degrees
- moved C34 7.82 mm to (242.0, 125.1), turned to 90 degrees
- moved C38 7.12 mm to (230.1, 134.3)
- moved U8 6.77 mm to (242.0, 132.8), turned to 90 degrees
- moved C35 4.34 mm to (230.1, 132.8)
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Connections:
- R18 pad 2: USB_R D+ -> Net-(U8-USB_DP)
- R19 pad 1: USB_R D- -> Net-(U8-USB_DM)
- S19 pad 1: GPIO_1_R -> GPIO_18_R
- S20 pad 1: GPIO_6_R -> GPIO_11_R
- S21 pad 1: GPIO_11_R -> GPIO_7_R
- S22 pad 1: GPIO_2_R -> GPIO_17_R
- S23 pad 1: GPIO_7_R -> GPIO_13_R
- S24 pad 1: GPIO_12_R -> GPIO_6_R
- S26 pad 1: GPIO_3_R -> GPIO_12_R
- S27 pad 1: GPIO_8_R -> GPIO_5_R
- S28 pad 1: GPIO_13_R -> GPIO_15_R
- S29 pad 1: GPIO_17_R -> GPIO_10_R
- S31 pad 1: GPIO_9_R -> GPIO_14_R
- S32 pad 1: GPIO_14_R -> GPIO_9_R
- S33 pad 1: GPIO_5_R -> GPIO_8_R
- S34 pad 1: GPIO_10_R -> GPIO_1_R
- S35 pad 1: GPIO_15_R -> GPIO_2_R
- S36 pad 1: GPIO_18_R -> GPIO_3_R
- U8 pad 30: R_TX -> R_RX
- U8 pad 31: R_RX -> R_TX
- U8 pad 46: USB_R D- -> Net-(U8-USB_DM)
- U8 pad 47: USB_R D+ -> Net-(U8-USB_DP)
Routing:
- net +3V3_R: track 88.7 -> 163.9 mm, vias 8 -> 14
- net GPIO_8_R: track 51.3 -> 113.9 mm, vias 1 -> 0
- net GPIO_15_R: track 36.6 -> 91.8 mm
- net GPIO_13_R: track 73.9 -> 31.9 mm, vias 1 -> 0
- net GPIO_5_R: track 111.3 -> 69.5 mm, vias 1 -> 0
- net GPIO_1_R: track 10.5 -> 49.2 mm, vias 1 -> 0
- net GPIO_6_R: track 12.6 -> 47.2 mm, vias 1 -> 0
- net GPIO_10_R: track 42.3 -> 75.9 mm
- net RESET_R: track 7.42 -> 38.2 mm, vias 0 -> 3
- net QSPI_SS_R: track 61.7 -> 34.5 mm, vias 3 -> 2
- net GPIO_17_R: track 69.5 -> 44.9 mm
- net GPIO_12_R: track 29.2 -> 53.0 mm, vias 1 -> 0
- net GPIO_11_R: track 34.6 -> 14.6 mm
- net GPIO_14_R: track 95.5 -> 115.2 mm, vias 1 -> 0
- net L_R D+: track 0.00 -> 18.5 mm
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- added copper zone on B.Cu, net +3V3_R
