File: PCBs/CustomKB2040.kicad_pcb (KiCad board)
At the start: 4 copper layers, 279 x 107 mm, 174 parts, among them J1 USB_C_Receptacle, J3 USB_C_Receptacle, J4 USB_C_Receptacle, J6 USB_C_Receptacle, U1 W25Q128JVS, U2 XC6206-3.3_SOT, U3 USBLC6-2SC6, U4 RP2040, U5 W25Q128JVS, U6 XC6206-3.3_SOT, U7 USBLC6-2SC6, U8 RP2040, Y1 Crystal_GND24, Y2 Crystal_GND24

Commit message: added library and routing changes
Parts:
- moved C30 0.70 mm to (230.8, 131.3)
- moved C35 0.69 mm to (230.8, 132.8)
- moved C38 0.69 mm to (230.8, 134.3)
- moved C3 0.10 mm to (165.5, 117.9)
- moved R5 0.10 mm to (164.0, 129.6)
- moved U1 0.10 mm to (166.5, 124.1)
Routing:
- net QSPI_SD3: track 16.2 -> 19.5 mm, vias 2 -> 0
- net QSPI_SCLK: track 14.4 -> 17.0 mm, vias 2 -> 0
- net GND: track 69.3 -> 68.0 mm, vias 59 -> 60
- net GND_R: track 63.0 -> 64.0 mm
- net +3V3_R: track 163.9 -> 164.7 mm
- net GPIO_11_R: vias 2 -> 1
- removed copper zone on B.Cu, net +3V3_R
Other:
- outline, holes or cut-outs redrawn
