File: PCBs/CustomKB2040.kicad_sch (KiCad schematic)
At the start: 0 parts

Commit message: mid way right side
Other:
- note added: "Both halves are identical. This is a split keyboard so there must be two PCBs, however for ease of manufacturing and file management I have them on the same "board" The notation "_R" is used to differitate between left and right mirrored elements -Jacob"
- note removed: "Both halves are identical. This is a split keyboard so there must be two PCBs, however for ease of manufacturing and file management I have them on the same "board" The notation "_R" is used to differitate between left and right mirrored elements -KQ4SPZ"
Changed lines of the file:
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@@
 		(comment 1 "SPARC")
 	)
-	(text "Both halves are identical. This is a split keyboard so there must be two PCBs,\nhowever for ease of manufacturing and file management I have them on the same \"board\"\nThe notation \"_R\" is used to differitate between left and right mirrored elements\n-KQ4SPZ"
+	(text "Both halves are identical. This is a split keyboard so there must be two PCBs,\nhowever for ease of manufacturing and file management I have them on the same \"board\"\nThe notation \"_R\" is used to differitate between left and right mirrored elements\n-Jacob"
 		(exclude_from_sim no)
 		(at 145.796 119.888 0)
